File: EAGLE/sr61/sr61-revC.brd (EAGLE design)
At the start: 283.8 x 93.2 mm, 220 parts, among them M1 M25C, X1 MICROMOD-2222-C

Commit message: ·
Parts:
- S1, S2: device VinoRodrigues_Custom_Eagle:SKRKAEE020 -> SilvinoR_Custom_Eagle:SKRKAEE020
Other:
- board text added: "(c) 2022 Silvino Rodrigues http://c1k.it/sr61"
- board text removed: "(c) 2022 Vino Rodrigues http://c1k.it/vr61"
Changed lines of the file:
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@@
 <wire x1="192.15" y1="7.85" x2="189.5" y2="7.85" width="1" layer="22"/>
 <text x="146.7046875" y="11.7203125" size="1.6764" layer="21" font="vector">tecsmith.com.au</text>
-<text x="138.3953125" y="19.9296875" size="1.6764" layer="21" font="vector" ratio="16">(c) 2022 Vino Rodrigues
-http://c1k.it/vr61</text>
+<text x="138.3953125" y="19.9296875" size="1.6764" layer="21" font="vector" ratio="16">(c) 2022 Silvino Rodrigues
+http://c1k.it/sr61</text>
 <text x="170.7" y="13" size="1.778" layer="21" rot="R270">BOOT</text>
 <text x="86.790625" y="14.1046875" size="1.6764" layer="21" font="vector">featuring</text>
 <text x="117.1" y="14.7" size="1.6764" layer="22" font="vector" rot="MR0">featuring</text>
-<text x="176.98125" y="12.8" size="1.6764" layer="22" font="vector" rot="MR0">(c) 2022 Vino Rodrigues
-http://c1k.it/vr61</text>
+<text x="176.98125" y="12.8" size="1.6764" layer="22" font="vector" rot="MR0">(c) 2022 Silvino Rodrigues
+http://c1k.it/sr61</text>
 <text x="168.2625" y="1.9" size="1.6764" layer="22" font="vector" rot="MR0">tecsmith.com.au</text>
 <text x="188.4" y="77.4" size="1" layer="26" rot="MR0" align="center-left">GND</text>
@@
 <text x="60.325" y="63.6" size="1.6764" layer="26" rot="MR0" align="center-right">!BOOT</text>
 <text x="59.125" y="63.575" size="1.6764" layer="26" rot="MR180" align="center-right">RESET</text>
-<text x="138.3953125" y="19.9296875" size="1.6764" layer="1" font="vector" ratio="16">(c) 2022 Vino Rodrigues
-http://c1k.it/vr61</text>
+<text x="138.3953125" y="19.9296875" size="1.6764" layer="1" font="vector" ratio="16">(c) 2022 Silvino Rodrigues
+http://c1k.it/sr61</text>
 <text x="106" y="64.77" size="1.35" layer="26" rot="MR0" align="bottom-center">1 2 3 4</text>
 <wire x1="148.59" y1="64.77" x2="160.02" y2="64.77" width="1" layer="26"/>
@@
 <element name="U$21" library="__temp_to_delete" package="FIDUCIAL" value="FIDUCIAL" x="259.525" y="92" smashed="yes"/>
 <element name="U$22" library="__temp_to_delete" package="FIDUCIAL" value="FIDUCIAL" x="283" y="50" smashed="yes"/>
-<element name="S1" library="VinoRodrigues_Custom_Eagle" package="SKRKAEE020" value="" x="58" y="60" smashed="yes" rot="MR90">
+<element name="S1" library="SilvinoR_Custom_Eagle" package="SKRKAEE020" value="" x="58" y="60" smashed="yes" rot="MR90">
 <attribute name="VALUE" x="53.19" y="56.62" size="1.778" layer="28" rot="MR90"/>
 </element>
-<element name="S2" library="VinoRodrigues_Custom_Eagle" package="SKRKAEE020" value="" x="61.45" y="60.025" smashed="yes" rot="MR90">
+<element name="S2" library="SilvinoR_Custom_Eagle" package="SKRKAEE020" value="" x="61.45" y="60.025" smashed="yes" rot="MR90">
 <attribute name="VALUE" x="56.64" y="56.645" size="1.778" layer="28" rot="MR90"/>
 </element>

Commit message: upgrades
Parts:
- added C15: 100nF, rcl:C0603
- added D69: (no value), jlcpcb_basic_parts:SOD-123
- added J-TTP: SM03B-SRSS-TB, __untitled:CONN_SM03B-SRSS-TB_JST
- added Q7: 2N7002, ts_custom_nick_nacks:SOT23-3
- added R32: 10K, rcl:R0603
- added TP1, TP2, TP3: TEST-POINT.3SQ, tecsmith_keyboards:PAD.03X.03-SQ
- added TTP223: (no value), tshome_touch:TTP223B
- turned T_ENT to 180 degrees
Connections:
- new net N$68: TP1.1, TTP223.6
- new net N$77: TP3.1, TTP223.4
- new net N$78: D69.A, Q7.2
- new net N$79: Q7.1, R32.1, TTP223.1
- new net N$80: J-TTP.2, J-TTP.3, TTP223.3
- net GND: now also C15.2, J-TTP.1, J-TTP.4, J-TTP.5, R32.2, TTP223.2
- net MX6: now also D69.C
- net MY8: now also Q7.3
- net VCC: now also C15.1, TP2.1, TTP223.5
Routing:
- net VCC: track 178.3 -> 277.2 mm, vias 12 -> 17
- net MY8: track 301.8 -> 351.3 mm, vias 6 -> 7
- net MX6: track 446.3 -> 482.6 mm, vias 15 -> 17
- net MY6: track 330.0 -> 313.4 mm
- net N$80: track 0.00 -> 1.57 mm
- net N$79: track 0.00 -> 1.37 mm
- net MX0: track 388.6 -> 387.8 mm
