File: EAGLE/sr61/sr61-revC.sch (EAGLE design)
At the start: 215 parts, among them M1 M25C, X1 MICROMOD-2222-C

Commit message: ·
Parts:
- S1, S2: device VinoRodrigues_Custom_Eagle:MOMENTARY-SWITCH-SPST-1 -> SilvinoR_Custom_Eagle:MOMENTARY-SWITCH-SPST-1
Changed lines of the file:
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@@
 <schematic xreflabel="%F%N/%S.%C%R" xrefpart="/%S.%C%R">
 <attributes>
-<attribute name="CNAME" value="VR61 - MicroMod 60% Custom Keyboard PCB"/>
+<attribute name="CNAME" value="SR61 - MicroMod 60% Custom Keyboard PCB"/>
 <attribute name="CREVISION" value="Rev A"/>
 </attributes>
@@
 <part name="U$21" library="__temp_to_delete" deviceset="FIDUCIAL" device=""/>
 <part name="U$22" library="__temp_to_delete" deviceset="FIDUCIAL" device=""/>
-<part name="S1" library="VinoRodrigues_Custom_Eagle" deviceset="MOMENTARY-SWITCH-SPST-1" device=""/>
-<part name="S2" library="VinoRodrigues_Custom_Eagle" deviceset="MOMENTARY-SWITCH-SPST-1" device=""/>
+<part name="S1" library="SilvinoR_Custom_Eagle" deviceset="MOMENTARY-SWITCH-SPST-1" device=""/>
+<part name="S2" library="SilvinoR_Custom_Eagle" deviceset="MOMENTARY-SWITCH-SPST-1" device=""/>
 <part name="C14" library="rcl" library_urn="urn:adsk.eagle:library:334" deviceset="C-EU" device="C0603" package3d_urn="urn:adsk.eagle:package:23616/2" value="100nF"/>
 <part name="D80" library="diode" library_urn="urn:adsk.eagle:library:210" deviceset="BAS70-05" device="" package3d_urn="urn:adsk.eagle:package:43389/2"/>

Commit message: upgrades
Parts:
- added C15: 100nF, rcl:C-EUC0603
- added D69: (no value), jlcpcb_basic_parts:1N5819WS
- added J-TTP: SM03B-SRSS-TB, __untitled:SM03B-SRSS-TB
- added Q7: 2N7002, ts_custom_nick_nacks:2N7002-BSS138
- added R32: 10K, rcl:R-EU_R0603
- added TP1, TP2, TP3: TEST-POINT.3SQ, tecsmith_keyboards:TEST-POINT.3SQ
- added TTP223: (no value), tshome_touch:TTP223-BA6
Connections:
- new net N$68: TP1.1, TTP223.P$6
- new net N$77: TP3.1, TTP223.P$4
- new net N$78: D69.A, Q7.S
- new net N$79: Q7.G, R32.1, TTP223.P$1
- new net N$80: J-TTP.2, J-TTP.3, TTP223.P$3
- net GND: now also C15.2, J-TTP.1, J-TTP.M, R32.2, TTP223.P$2
- net MX6: now also D69.C
- net MY8: now also Q7.D
- net VCC: now also C15.1, TP2.1, TTP223.P$5
Other:
- note added: "Optional (Touch) **DNP**"
- moved on the sheet: H5, J-52, J-63, J-UDB, JP-GND
